File: voz-9/kicad/voz-9.kicad_pcb (KiCad board)
At the start: 2 copper layers, 300 x 300 mm, 189 parts, among them J1 OSC, J2 LFO, J3 DELAY, J4 PATCH A, J5 PATCH B, J6 CTRL, J7 IN+PRE, J8 OUT, J9 EQ424, Q1 J201, Q2 J201, Q3 J201, Q4 J201, Q5 J201, Q6 J201, Q7 2N5457, U1 NE5532, U2 TL072, U3 TL072, U4 MAX1044, U5 78M05, U6 PT2399, U7 PT2399, U8 PT2399, U9 TL072

Commit message: Espalha os blocos na BASE e troca J1–J9 por pinos 1×N na borda de baixo.
O circuito deixa o bloco central de 220×160 e ocupa a placa de 300×300 por faixas, com folga para solda. Os conectores do painel na placa passam de soquete fêmea 2×N para barra de pinos macho; o fio solda na base.

Co-authored-by: Andrey <andreysenes@users.noreply.github.com>
Parts:
- J1, J3, J4: footprint voz9:PinSocket_2x10_TopBottom -> Connector_PinHeader_2.54mm:PinHeader_1x20_P2.54mm_Vertical
- J2, J7, J9: footprint voz9:PinSocket_2x06_TopBottom -> Connector_PinHeader_2.54mm:PinHeader_1x12_P2.54mm_Vertical
- J5: footprint voz9:PinSocket_2x08_TopBottom -> Connector_PinHeader_2.54mm:PinHeader_1x16_P2.54mm_Vertical
- J6, J8: footprint voz9:PinSocket_2x03_TopBottom -> Connector_PinHeader_2.54mm:PinHeader_1x06_P2.54mm_Vertical
- moved J5 225.2 mm to (241.9, 293.0), turned to 90 degrees
- moved R9 216.8 mm to (15.2, 177.4)
- moved R10 213.3 mm to (29.0, 177.4)
- moved J1 210.1 mm to (16.0, 293.0), turned to 90 degrees
- moved D3 208.6 mm to (15.5, 170.0)
- moved D4 206.3 mm to (29.8, 170.0)
- moved C70 205.5 mm to (37.5, 252.4)
- moved J8 204.9 mm to (267.3, 283.5), turned to 90 degrees
- moved R59 204.3 mm to (43.8, 170.0)
- moved C69 203.4 mm to (27.7, 252.4)
- moved C42 198.0 mm to (15.5, 251.2)
- moved R60 196.5 mm to (42.8, 177.4)
- moved J6 187.6 mm to (215.9, 283.5), turned to 90 degrees
- moved J4 183.3 mm to (166.6, 293.0), turned to 90 degrees
- moved J2 179.2 mm to (16.0, 283.5), turned to 90 degrees
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Other:
- board text added: "CLK"
- board text added: "ENV"
- board text added: "FITA"
- board text added: "FONTE"
- board text added: "J1 OSC"
- board text added: "J2 LFO"
- board text added: "J3 DELAY"
- board text added: "J4 PATCH A"
- board text added: "J5 PATCH B"
- board text added: "J6 CTRL"
- board text added: "J7 IN+PRE"
- board text added: "J8 OUT"
- board text added: "J9 EQ424"
- board text added: "MIX"
- board text added: "NAB"
- board text added: "TRIM"
- board text added: "U1"
- board text added: "U2"
- board text added: "VCF"
- board text added: "fio na base, pinos 1xN pino 1 a esquerda de cada grupo CIs em soquete cobre no verso"
- board text removed: "4V5"
- board text removed: "GND"
- board text removed: "V9"
- board text removed: "miolo 220x160 centrado cobre no verso CIs em soquete pino 1 quadrado nos J"

Commit message: Agrupa a BASE pelo sinal para encurtar trilha e jumper.
Cada bloco fica junto do conector que o serve, com corredor de alimentação em cima e de áudio no meio. O 1N5817 aponta para J6, o oscilador senta em J1 e o pré em J7. O esquema repete esses blocos, ainda sem fios.

Co-authored-by: Andrey <andreysenes@users.noreply.github.com>
Parts:
- moved R63 334.0 mm to (15.2, 243.0)
- moved D1 288.1 mm to (224.0, 250.0), turned to -90 degrees
- moved R62 286.1 mm to (62.2, 236.6)
- moved R22 285.4 mm to (49.4, 236.6)
- moved R21 284.7 mm to (36.6, 236.6)
- moved U2 278.6 mm to (15.8, 222.2)
- moved R72 273.7 mm to (28.0, 243.0)
- moved R32 273.1 mm to (15.2, 199.6)
- moved R61 263.5 mm to (28.0, 193.2)
- moved R67 262.5 mm to (15.2, 193.2)
- moved C19 256.8 mm to (67.9, 222.0)
- moved C6 256.1 mm to (57.2, 222.0)
- moved C21 255.4 mm to (46.5, 222.0)
- moved C44 255.0 mm to (26.2, 186.8)
- moved C43 254.0 mm to (15.5, 186.8)
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Other:
- board text added: "EQ"
- board text added: "EQ 424"
- board text added: "MOD"
- board text added: "OSC"
- board text added: "OUT"
- board text added: "PRE"
- board text added: "barramento V9 GND VEE V5 4V5 1V8"
- board text added: "canal de audio"
- board text added: "fio na base, pino 1 a esquerda cobre no verso corredores livres para o barramento e o audio"
- board text removed: "ENV"
- board text removed: "TRIM"
- board text removed: "U1"
- board text removed: "U2"
- board text removed: "VCF"
- board text removed: "fio na base, pinos 1xN pino 1 a esquerda de cada grupo CIs em soquete cobre no verso"
