File: voz-9/kicad/voz-9.kicad_pcb (KiCad board)
At the start: 2 copper layers, 300 x 300 mm, 189 parts, among them J1 OSC, J2 LFO, J3 DELAY, J4 PATCH A, J5 PATCH B, J6 CTRL, J7 IN+PRE, J8 OUT, J9 EQ424, Q1 J201, Q2 J201, Q3 J201, Q4 J201, Q5 J201, Q6 J201, Q7 2N5457, U1 NE5532, U2 TL072, U3 TL072, U4 MAX1044, U5 78M05, U6 PT2399, U7 PT2399, U8 PT2399, U9 TL072

Commit message: Roteia a BASE nas duas faces e fecha o plano de GND no verso.
As nets seguem o circuito do esquema. O cobre passa no DRC: trilhas ligadas, sem folga violada. O pino 1 dos JFET fica redondo para o TO-92 caber na folga de 0,35 mm.

Co-authored-by: Andrey <andreysenes@users.noreply.github.com>
Connections:
- C1 pad 1: (no net) -> XLR_HOT
- C1 pad 2: (no net) -> GND
- C10 pad 1: (no net) -> U6_LP1
- C10 pad 2: (no net) -> GND
- C11 pad 1: (no net) -> U7_LP1
- C11 pad 2: (no net) -> GND
- C12 pad 1: (no net) -> U8_LP1
- C12 pad 2: (no net) -> GND
- C13 pad 1: (no net) -> U6_OP
- C13 pad 2: (no net) -> U6_OUT
- C14 pad 1: (no net) -> U7_OP
- C14 pad 2: (no net) -> U7_OUT
- C15 pad 1: (no net) -> U8_OP
- C15 pad 2: (no net) -> U8_OUT
- C16 pad 1: (no net) -> U6_LP1
- C16 pad 2: (no net) -> GND
- C17 pad 1: (no net) -> U7_LP1
- C17 pad 2: (no net) -> GND
- C18 pad 1: (no net) -> U8_LP1
- C18 pad 2: (no net) -> GND
- C19 pad 1: (no net) -> V9
- C19 pad 2: (no net) -> GND
- C2 pad 1: (no net) -> XLR_COLD
- C2 pad 2: (no net) -> GND
- C20 pad 1: (no net) -> U3A_OUT
- C20 pad 2: (no net) -> HEADS
- C21 pad 1: (no net) -> U2A_INM
- C21 pad 2: (no net) -> N4V5
- C22 pad 1: (no net) -> V5
- C22 pad 2: (no net) -> GND
- C23 pad 1: (no net) -> V9
- C23 pad 2: (no net) -> GND
- C24 pad 1: (no net) -> VEE
- C24 pad 2: (no net) -> GND
- C25 pad 1: (no net) -> U1_OA
- C25 pad 2: (no net) -> U1_BP
- C26 pad 1: (no net) -> NOISE_D
- C26 pad 2: (no net) -> NOISE_MIX
- C27 pad 1: (no net) -> PRE_W
- C27 pad 2: (no net) -> FALA
- C28 pad 1: (no net) -> SHAPE
- C28 pad 2: (no net) -> FILT_SW
- C29 pad 1: (no net) -> WET_MIX
- C29 pad 2: (no net) -> LE_IN
- C3 pad 1: (no net) -> WET_LP
- C3 pad 2: (no net) -> GND
- C30 pad 1: (no net) -> MIX
- C30 pad 2: (no net) -> EQ_IN
- C31 pad 1: (no net) -> V5
- C31 pad 2: (no net) -> GND
- C32 pad 1: (no net) -> V5
- C32 pad 2: (no net) -> GND
- C33 pad 1: (no net) -> V5
- C33 pad 2: (no net) -> GND
- C34 pad 1: (no net) -> U6_OUT
- C34 pad 2: (no net) -> U6_SW
- C35 pad 1: (no net) -> U7_OUT
- C35 pad 2: (no net) -> U7_SW
- C36 pad 1: (no net) -> U8_OUT
- C36 pad 2: (no net) -> U8_SW
- C37 pad 1: (no net) -> PT_REF_U6
- C37 pad 2: (no net) -> GND
- C38 pad 1: (no net) -> PT_REF_U7
- C38 pad 2: (no net) -> GND
- C39 pad 1: (no net) -> PT_REF_U8
- C39 pad 2: (no net) -> GND
- C4 pad 1: (no net) -> U3A_IN
- C4 pad 2: (no net) -> U3A_OUT
- C40 pad 1: (no net) -> V9
- C40 pad 2: (no net) -> GND
- C41 pad 1: (no net) -> PRE_W
- C41 pad 2: (no net) -> OSCIN_CW
- C42 pad 1: (no net) -> U1_OB
- C42 pad 2: (no net) -> PRE_CW
- C43 pad 1: (no net) -> LFO_D
- C43 pad 2: (no net) -> LFO_N1
- C44 pad 1: (no net) -> LFO_N1
- C44 pad 2: (no net) -> LFO_N2
- C45 pad 1: (no net) -> INST_TIP
- C45 pad 2: (no net) -> EXT_IN
- C46 pad 1: (no net) -> TREM_A
- C46 pad 2: (no net) -> LFO_G
- C47 pad 1: (no net) -> VCF
- C47 pad 2: (no net) -> GND
- C48 pad 1: (no net) -> GRAVA_IN
- C48 pad 2: (no net) -> NAB_MID
- C49 pad 1: (no net) -> NAB_BASS
- C49 pad 2: (no net) -> WET
- C5 pad 1: (no net) -> U3B_IN
- C5 pad 2: (no net) -> WET
- C50 pad 1: (no net) -> VCF
- C50 pad 2: (no net) -> VCA_D
- C51 pad 1: (no net) -> U2A_OUT
- C51 pad 2: (no net) -> SW_A
- C52 pad 1: (no net) -> U2B_OUT
- C52 pad 2: (no net) -> SW_B
- C53 pad 1: (no net) -> LFO_D
- C53 pad 2: (no net) -> LFO_AC
- C54 pad 1: (no net) -> VCA_S
- C54 pad 2: (no net) -> DRY
- C55 pad 1: (no net) -> CLK_B
- C55 pad 2: (no net) -> GND
- C56 pad 1: (no net) -> U4_CAP+
- C56 pad 2: (no net) -> U4_CAP-
- C57 pad 1: (no net) -> VEE
- C57 pad 2: (no net) -> GND
- C58 pad 1: (no net) -> V5
- C58 pad 2: (no net) -> GND
- C59 pad 1: (no net) -> XLR_HOT
- C59 pad 2: (no net) -> PRE_R12
- C6 pad 1: (no net) -> U2B_INM
- C6 pad 2: (no net) -> N4V5
- C60 pad 1: (no net) -> XLR_COLD
- C60 pad 2: (no net) -> PRE_R13
- C61 pad 1: (no net) -> V9
- C61 pad 2: (no net) -> GND
- C62 pad 1: (no net) -> VEE
- C62 pad 2: (no net) -> GND
- C63 pad 1: (no net) -> V5
- C63 pad 2: (no net) -> GND
- C64 pad 1: (no net) -> V9
- C64 pad 2: (no net) -> GND
- C65 pad 1: (no net) -> VEE
- C65 pad 2: (no net) -> GND
- C66 pad 1: (no net) -> N4V5
- C66 pad 2: (no net) -> GND
- C67 pad 1: (no net) -> N1V8
- C67 pad 2: (no net) -> GND
- C68 pad 1: (no net) -> ENV
- C68 pad 2: (no net) -> GND
- C69 pad 1: (no net) -> U7_OUT
- C69 pad 2: (no net) -> U7_SW
- C7 pad 1: (no net) -> U6_CC1
- C7 pad 2: (no net) -> U6_CC0
- C70 pad 1: (no net) -> U8_OUT
- C70 pad 2: (no net) -> U8_SW
- C71 pad 1: (no net) -> TREM_B
- C71 pad 2: (no net) -> LFO_G
- C8 pad 1: (no net) -> U7_CC1
- C8 pad 2: (no net) -> U7_CC0
- C9 pad 1: (no net) -> U8_CC1
- C9 pad 2: (no net) -> U8_CC0
- D1 pad 1: (no net) -> V9
- D1 pad 2: (no net) -> P4_TIP
- D2 pad 1: (no net) -> ENV
- D2 pad 2: (no net) -> GATE
- D3 pad 1: (no net) -> ENV
- D3 pad 2: (no net) -> FALA_A
- D4 pad 1: (no net) -> CLK_B
- D4 pad 2: (no net) -> CLK_A
- D6 pad 1: (no net) -> GND
- D6 pad 2: (no net) -> SHAPE
- D7 pad 1: (no net) -> GND
- D7 pad 2: (no net) -> WET
- J1 pad 1: (no net) -> OSC_A_POT
- J1 pad 10: (no net) -> GND
- J1 pad 11: (no net) -> N1V8
- J1 pad 12: (no net) -> CUT_W
- J1 pad 13: (no net) -> GND
- J1 pad 14: (no net) -> SW_A
- J1 pad 15: (no net) -> SW_A_ON
- J1 pad 16: (no net) -> SW_B
- J1 pad 17: (no net) -> SW_B_ON
- J1 pad 18: (no net) -> N1V8
- J1 pad 19: (no net) -> ENV
- J1 pad 2: (no net) -> U2A_INM
- J1 pad 3: (no net) -> OSC_B_POT
- J1 pad 4: (no net) -> U2B_INM
- J1 pad 5: (no net) -> SUM
- J1 pad 6: (no net) -> AMT_W
- J1 pad 7: (no net) -> GND
- J1 pad 8: (no net) -> EQ_OUT
- J1 pad 9: (no net) -> SHAPE_W
- J2 pad 1: (no net) -> RATE_W
- J2 pad 10: (no net) -> DEPTH_W
- J2 pad 11: (no net) -> PITCH_CV
- J2 pad 12: (no net) -> TIME_CV
- J2 pad 2: (no net) -> RATE_W
- J2 pad 3: (no net) -> GND
- J2 pad 4: (no net) -> LFO_OUT
- J2 pad 5: (no net) -> DEPTH_W
- J2 pad 6: (no net) -> GND
- J2 pad 7: (no net) -> LFO_N2
- J2 pad 8: (no net) -> TREM_A
- J2 pad 9: (no net) -> TREM_B
- J3 pad 1: (no net) -> V5
- J3 pad 10: (no net) -> GND
- J3 pad 11: (no net) -> STAR
- J3 pad 12: (no net) -> FB_CW
- J3 pad 13: (no net) -> DRY
- J3 pad 14: (no net) -> WET_W
- J3 pad 15: (no net) -> WET
- J3 pad 16: (no net) -> U6_SW
- J3 pad 17: (no net) -> U7_IN
- J3 pad 18: (no net) -> GND
- J3 pad 19: (no net) -> OUT
- J3 pad 2: (no net) -> TIME_W
- J3 pad 20: (no net) -> WET_W
- J3 pad 3: (no net) -> GND
- J3 pad 4: (no net) -> U6_SW
- J3 pad 5: (no net) -> H1_ON
- J3 pad 6: (no net) -> U7_SW
- J3 pad 7: (no net) -> H2_ON
- J3 pad 8: (no net) -> U8_SW
- J3 pad 9: (no net) -> H3_ON
- J4 pad 1: (no net) -> SW_A_ON
- J4 pad 10: (no net) -> FILT_TIP
- J4 pad 11: (no net) -> FILT_SW
- J4 pad 12: (no net) -> GND
- J4 pad 13: (no net) -> FCV
- J4 pad 15: (no net) -> GND
- J4 pad 16: (no net) -> VCV
- J4 pad 18: (no net) -> GND
- J4 pad 3: (no net) -> GND
- J4 pad 4: (no net) -> SW_B_ON
- J4 pad 6: (no net) -> GND
- J4 pad 7: (no net) -> EXT_IN
- J4 pad 9: (no net) -> GND
- J5 pad 1: (no net) -> LFO_OUT
- J5 pad 10: (no net) -> PRE_W
- J5 pad 12: (no net) -> GND
- J5 pad 13: (no net) -> STAR
- J5 pad 14: (no net) -> PRE_W
- J5 pad 15: (no net) -> GND
- J5 pad 3: (no net) -> GND
- J5 pad 4: (no net) -> TIME_CV
- J5 pad 6: (no net) -> GND
- J5 pad 7: (no net) -> CLK_TIP
- J5 pad 9: (no net) -> GND
- J6 pad 1: (no net) -> LED_A
- J6 pad 2: (no net) -> GND
- J6 pad 3: (no net) -> P4_TIP
- J6 pad 4: (no net) -> GND
- J6 pad 5: (no net) -> GATE
- J6 pad 6: (no net) -> GND
- J7 pad 1: (no net) -> XLR_HOT
- J7 pad 10: (no net) -> MIX
- J7 pad 11: (no net) -> OSCIN_CW
- J7 pad 2: (no net) -> XLR_COLD
- J7 pad 3: (no net) -> GND
- J7 pad 4: (no net) -> INST_TIP
- J7 pad 5: (no net) -> GND
- J7 pad 6: (no net) -> GND
- J7 pad 7: (no net) -> PRE_W
- J7 pad 8: (no net) -> PRE_CW
- J7 pad 9: (no net) -> AMT_W
- J8 pad 1: (no net) -> XLR_OUT
- J8 pad 2: (no net) -> J8_COLD
- J8 pad 3: (no net) -> GND
- J8 pad 4: (no net) -> OUT
- J8 pad 5: (no net) -> GND
- Q1 pad 1: (no net) -> U2A_INM
- Q1 pad 2: (no net) -> Q1G
- Q1 pad 3: (no net) -> N4V5
- Q2 pad 1: (no net) -> U2B_INM
- Q2 pad 2: (no net) -> Q2G
- Q2 pad 3: (no net) -> N4V5
- Q3 pad 1: (no net) -> NOISE_D
- Q3 pad 2: (no net) -> Q3G
- Q3 pad 3: (no net) -> NOISE_S
- Q4 pad 1: (no net) -> VCF
- Q4 pad 2: (no net) -> Q4G
- Q4 pad 3: (no net) -> N1V8
- Q5 pad 1: (no net) -> VCA_D
- Q5 pad 2: (no net) -> ENV
- Q5 pad 3: (no net) -> VCA_S
- Q6 pad 1: (no net) -> V9
- Q6 pad 2: (no net) -> Q6G
- Q6 pad 3: (no net) -> Q6S
- Q7 pad 1: (no net) -> LFO_D
- Q7 pad 2: (no net) -> LFO_G
- Q7 pad 3: (no net) -> LFO_S
- R1 pad 1: (no net) -> XLR_OUT
- R1 pad 2: (no net) -> GND
- R10 pad 1: (no net) -> H3A
- R10 pad 2: (no net) -> H3B
- R11 pad 1: (no net) -> TIME_W
- R11 pad 2: (no net) -> PT6_U6
- R12 pad 1: (no net) -> PRE_R12
- R12 pad 2: (no net) -> U1_INP
- R13 pad 1: (no net) -> PRE_R13
- R13 pad 2: (no net) -> U1_INM
- R14 pad 1: (no net) -> V9
- R14 pad 2: (no net) -> LED_A
- R15 pad 1: (no net) -> LFO_G
- R15 pad 2: (no net) -> RATE_W
- R16 pad 1: (no net) -> NAB_MID
- R16 pad 2: (no net) -> U3A_IN
- R18 pad 1: (no net) -> N1V8
- R18 pad 2: (no net) -> GND
- R19 pad 1: (no net) -> V9
- R19 pad 2: (no net) -> N4V5
- R2 pad 1: (no net) -> J8_COLD
- R2 pad 2: (no net) -> GND
- R20 pad 1: (no net) -> N4V5
- R20 pad 2: (no net) -> GND
- R21 pad 1: (no net) -> U2A_OUT
- R21 pad 2: (no net) -> OSC_A_POT
- R22 pad 1: (no net) -> U2B_OUT
- R22 pad 2: (no net) -> OSC_B_POT
- R23 pad 1: (no net) -> V9
- R23 pad 2: (no net) -> NOISE_D
- R24 pad 1: (no net) -> SW_A_ON
- R24 pad 2: (no net) -> SUM
- R25 pad 1: (no net) -> SW_B_ON
- R25 pad 2: (no net) -> SUM
- R26 pad 1: (no net) -> EXT_IN
- R26 pad 2: (no net) -> SUM
- R27 pad 1: (no net) -> EQ_OUT
- R27 pad 2: (no net) -> Q6G
- R28 pad 1: (no net) -> Q6S
- R28 pad 2: (no net) -> SHAPE
- R29 pad 1: (no net) -> SHAPE_W
- R29 pad 2: (no net) -> SHAPE
- R3 pad 1: (no net) -> NOISE_S
- R3 pad 2: (no net) -> GND
- R30 pad 1: (no net) -> FILT_TIP
- R30 pad 2: (no net) -> VCF
- R31 pad 1: (no net) -> V9
- R31 pad 2: (no net) -> LFO_D
- R32 pad 1: (no net) -> LFO_N1
- R32 pad 2: (no net) -> GND
- R33 pad 1: (no net) -> LFO_N2
- R33 pad 2: (no net) -> GND
- R34 pad 1: (no net) -> VCA_S
- R34 pad 2: (no net) -> N1V8
- R35 pad 1: (no net) -> HEADS
- R35 pad 2: (no net) -> U6_IN
- R36 pad 1: (no net) -> HEADS
- R36 pad 2: (no net) -> U7_IN
- R37 pad 1: (no net) -> HEADS
- R37 pad 2: (no net) -> U8_IN
- R38 pad 1: (no net) -> H1_ON
- R38 pad 2: (no net) -> WET_MIX
- R39 pad 1: (no net) -> H2_ON
- R39 pad 2: (no net) -> WET_MIX
- R4 pad 1: (no net) -> Q6S
- R4 pad 2: (no net) -> N4V5
- R40 pad 1: (no net) -> H3_ON
- R40 pad 2: (no net) -> WET_MIX
- R41 pad 1: (no net) -> U6_IN
- R41 pad 2: (no net) -> U6_LP1
- R42 pad 1: (no net) -> U1_BM
- R42 pad 2: (no net) -> U1_OB
- R43 pad 1: (no net) -> CLK_A
- R43 pad 2: (no net) -> GND
- R44 pad 1: (no net) -> OUT
- R44 pad 2: (no net) -> XLR_OUT
- R45 pad 1: (no net) -> U3B_IN
- R45 pad 2: (no net) -> NAB_BASS
- R46 pad 1: (no net) -> DRY
- R46 pad 2: (no net) -> STAR
- R47 pad 1: (no net) -> U7_IN
- R47 pad 2: (no net) -> U7_LP1
- R48 pad 1: (no net) -> U8_IN
- R48 pad 2: (no net) -> U8_LP1
- R49 pad 1: (no net) -> WET
- R49 pad 2: (no net) -> WET_LP
- R5 pad 1: (no net) -> LFO_S
- R5 pad 2: (no net) -> GND
- R50 pad 1: (no net) -> FALA
- R50 pad 2: (no net) -> FALA_A
- R51 pad 1: (no net) -> STAR
- R51 pad 2: (no net) -> GRAVA_IN
- R52 pad 1: (no net) -> U3A_IN
- R52 pad 2: (no net) -> U3A_OUT
- R53 pad 1: (no net) -> LE_IN
- R53 pad 2: (no net) -> U3B_IN
- R54 pad 1: (no net) -> U3B_IN
- R54 pad 2: (no net) -> WET
- R55 pad 1: (no net) -> V9
- R55 pad 2: (no net) -> N1V8
- R56 pad 1: (no net) -> H2B
- R56 pad 2: (no net) -> PT6_U7
- R57 pad 1: (no net) -> U1_INM
- R57 pad 2: (no net) -> U1_OA
- R58 pad 1: (no net) -> U1_INP
- R58 pad 2: (no net) -> GND
- R59 pad 1: (no net) -> CLK_TIP
- R59 pad 2: (no net) -> CLK_A
- R6 pad 1: (no net) -> U1_BM
- R6 pad 2: (no net) -> GND
- R60 pad 1: (no net) -> H3B
- R60 pad 2: (no net) -> PT6_U8
- R61 pad 1: (no net) -> VCF
- R61 pad 2: (no net) -> RES_W
- R62 pad 1: (no net) -> U2A_OUT
- R62 pad 2: (no net) -> U2A_INP
- R63 pad 1: (no net) -> U2A_INP
- R63 pad 2: (no net) -> N4V5
- R64 pad 1: (no net) -> NOISE_MIX
- R64 pad 2: (no net) -> SUM
- R65 pad 1: (no net) -> PITCH_CV
- R65 pad 2: (no net) -> Q1G
- R66 pad 1: (no net) -> PITCH_CV
- R66 pad 2: (no net) -> Q2G
- R67 pad 1: (no net) -> Q4G
- R67 pad 2: (no net) -> FCV
- R68 pad 1: (no net) -> CUT_W
- R68 pad 2: (no net) -> Q4G
- R69 pad 1: (no net) -> ENV
- R69 pad 2: (no net) -> VCV
- R7 pad 1: (no net) -> TIME_W
- R7 pad 2: (no net) -> H2A
- R70 pad 1: (no net) -> CLK_B
- R70 pad 2: (no net) -> TIME_CV
- R71 pad 1: (no net) -> WET
- R71 pad 2: (no net) -> WET_W
- R72 pad 1: (no net) -> U2B_OUT
- R72 pad 2: (no net) -> U2B_INP
- R73 pad 1: (no net) -> U2B_INP
- R73 pad 2: (no net) -> N4V5
- R74 pad 1: (no net) -> ENV
- R74 pad 2: (no net) -> GND
- R75 pad 1: (no net) -> TIME_CV
- R75 pad 2: (no net) -> PT6_U6
- R76 pad 1: (no net) -> TIME_CV
- R76 pad 2: (no net) -> PT6_U7
- R77 pad 1: (no net) -> TIME_CV
- R77 pad 2: (no net) -> PT6_U8
- R78 pad 1: (no net) -> CLK_B
- R78 pad 2: (no net) -> GND
- R79 pad 1: (no net) -> LFO_AC
- R79 pad 2: (no net) -> LFO_OUT
- R8 pad 1: (no net) -> H2A
- R8 pad 2: (no net) -> H2B
- R80 pad 1: (no net) -> Q3G
- R80 pad 2: (no net) -> GND
- R81 pad 1: (no net) -> LFO_G
- R81 pad 2: (no net) -> GND
- R9 pad 1: (no net) -> TIME_W
- R9 pad 2: (no net) -> H3A
- RV1 pad 1: (no net) -> WET
- RV1 pad 2: (no net) -> FB_CW
- RV1 pad 3: (no net) -> FB_CW
- RV2 pad 1: (no net) -> FILT_TIP
- RV2 pad 2: (no net) -> RES_W
- RV2 pad 3: (no net) -> FILT_TIP
- U1 pad 1: (no net) -> U1_OA
- U1 pad 2: (no net) -> U1_INM
- U1 pad 3: (no net) -> U1_INP
- U1 pad 4: (no net) -> VEE
- U1 pad 5: (no net) -> U1_BP
- U1 pad 6: (no net) -> U1_BM
- U1 pad 7: (no net) -> U1_OB
- U1 pad 8: (no net) -> V9
- U2 pad 1: (no net) -> U2A_OUT
- U2 pad 2: (no net) -> U2A_INM
- U2 pad 3: (no net) -> U2A_INP
- U2 pad 4: (no net) -> GND
- U2 pad 5: (no net) -> U2B_INP
- U2 pad 6: (no net) -> U2B_INM
- U2 pad 7: (no net) -> U2B_OUT
- U2 pad 8: (no net) -> V9
- U3 pad 1: (no net) -> U3A_OUT
- U3 pad 2: (no net) -> U3A_IN
- U3 pad 3: (no net) -> GND
- U3 pad 4: (no net) -> VEE
- U3 pad 5: (no net) -> GND
- U3 pad 6: (no net) -> U3B_IN
- U3 pad 7: (no net) -> WET
- U3 pad 8: (no net) -> V9
- U4 pad 2: (no net) -> U4_CAP+
- U4 pad 3: (no net) -> GND
- U4 pad 4: (no net) -> U4_CAP-
- U4 pad 5: (no net) -> VEE
- U4 pad 8: (no net) -> V9
- U5 pad 1: (no net) -> V9
- U5 pad 2: (no net) -> GND
- U5 pad 3: (no net) -> V5
- U6 pad 1: (no net) -> V5
- U6 pad 10: (no net) -> U6_OP
- U6 pad 11: (no net) -> U6_OP
- U6 pad 12: (no net) -> U6_OP
- U6 pad 13: (no net) -> U6_OP
- U6 pad 14: (no net) -> U6_OUT
- U6 pad 15: (no net) -> U6_LP1
- U6 pad 16: (no net) -> U6_IN
- U6 pad 2: (no net) -> PT_REF_U6
- U6 pad 3: (no net) -> GND
- U6 pad 4: (no net) -> GND
- U6 pad 6: (no net) -> PT6_U6
- U6 pad 7: (no net) -> U6_CC1
- U6 pad 8: (no net) -> U6_CC0
- U6 pad 9: (no net) -> U6_OP
- U7 pad 1: (no net) -> V5
- U7 pad 10: (no net) -> U7_OP
- U7 pad 11: (no net) -> U7_OP
- U7 pad 12: (no net) -> U7_OP
- U7 pad 13: (no net) -> U7_OP
- U7 pad 14: (no net) -> U7_OUT
- U7 pad 15: (no net) -> U7_LP1
- U7 pad 16: (no net) -> U7_IN
- U7 pad 2: (no net) -> PT_REF_U7
- U7 pad 3: (no net) -> GND
- U7 pad 4: (no net) -> GND
- U7 pad 6: (no net) -> PT6_U7
- U7 pad 7: (no net) -> U7_CC1
- U7 pad 8: (no net) -> U7_CC0
- U7 pad 9: (no net) -> U7_OP
- U8 pad 1: (no net) -> V5
- U8 pad 10: (no net) -> U8_OP
- U8 pad 11: (no net) -> U8_OP
- U8 pad 12: (no net) -> U8_OP
- U8 pad 13: (no net) -> U8_OP
- U8 pad 14: (no net) -> U8_OUT
- U8 pad 15: (no net) -> U8_LP1
- U8 pad 16: (no net) -> U8_IN
- U8 pad 2: (no net) -> PT_REF_U8
- U8 pad 3: (no net) -> GND
- U8 pad 4: (no net) -> GND
- U8 pad 6: (no net) -> PT6_U8
- U8 pad 7: (no net) -> U8_CC1
- U8 pad 8: (no net) -> U8_CC0
- U8 pad 9: (no net) -> U8_OP
- U9 pad 1: (no net) -> EQ_A
- U9 pad 2: (no net) -> EQ_A
- U9 pad 3: (no net) -> EQ_IN
- U9 pad 4: (no net) -> VEE
- U9 pad 5: (no net) -> EQ_A
- U9 pad 6: (no net) -> EQ_OUT
- U9 pad 7: (no net) -> EQ_OUT
- U9 pad 8: (no net) -> V9
Routing:
- net GND: track 0.00 -> 1576.4 mm, vias 0 -> 2
- net V9: track 0.00 -> 902.1 mm, vias 0 -> 2
- net V5: track 0.00 -> 636.2 mm, vias 0 -> 3
- net N1V8: track 0.00 -> 482.9 mm, vias 0 -> 1
- net TIME_CV: track 0.00 -> 459.4 mm, vias 0 -> 6
- net N4V5: track 0.00 -> 433.8 mm, vias 0 -> 2
- net PRE_W: track 0.00 -> 398.0 mm, vias 0 -> 4
- net EQ_OUT: track 0.00 -> 385.8 mm
- net OUT: track 0.00 -> 373.0 mm
- net WET: track 0.00 -> 359.4 mm, vias 0 -> 1
- net VEE: track 0.00 -> 357.3 mm
- net U7_SW: track 0.00 -> 339.8 mm, vias 0 -> 1
- net SUM: track 0.00 -> 328.6 mm, vias 0 -> 1
- net EXT_IN: track 0.00 -> 326.9 mm, vias 0 -> 2
- net SW_B_ON: track 0.00 -> 323.0 mm, vias 0 -> 1
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- added copper zone on B.Cu, net GND

Commit message: Encolhe a BASE para 300×140 mm e reagrupa os blocos.
Duas placas cabem numa chapa de 300×300. Cada bloco fica junto do pino, o pino 1 do TO-92 fica redondo e a folha acompanha o contorno.

Co-authored-by: Andrey <andreysenes@users.noreply.github.com>
Parts:
- moved Q3 248.1 mm to (253.8, 45.2)
- moved Q6 247.9 mm to (262.2, 45.2)
- moved D6 247.7 mm to (270.3, 44.0)
- moved R27 243.5 mm to (253.2, 70.4)
- moved R28 243.3 mm to (265.8, 70.4)
- moved R4 243.1 mm to (278.4, 70.4)
- moved D1 235.8 mm to (194.9, 16.0), turned to 0 degrees
- moved C26 216.6 mm to (253.5, 51.8)
- moved R23 216.4 mm to (263.7, 51.8)
- moved R24 216.2 mm to (276.3, 51.8)
- moved R65 204.7 mm to (253.2, 76.6)
- moved R66 204.5 mm to (265.8, 76.6)
- moved R73 204.3 mm to (278.4, 76.6)
- moved R47 194.2 mm to (134.4, 85.0)
- moved R41 194.0 mm to (121.8, 85.0)
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Connections:
- C1 pad 1: XLR_HOT -> (no net)
- C1 pad 2: GND -> (no net)
- C10 pad 1: U6_LP1 -> (no net)
- C10 pad 2: GND -> (no net)
- C11 pad 1: U7_LP1 -> (no net)
- C11 pad 2: GND -> (no net)
- C12 pad 1: U8_LP1 -> (no net)
- C12 pad 2: GND -> (no net)
- C13 pad 1: U6_OP -> (no net)
- C13 pad 2: U6_OUT -> (no net)
- C14 pad 1: U7_OP -> (no net)
- C14 pad 2: U7_OUT -> (no net)
- C15 pad 1: U8_OP -> (no net)
- C15 pad 2: U8_OUT -> (no net)
- C16 pad 1: U6_LP1 -> (no net)
- C16 pad 2: GND -> (no net)
- C17 pad 1: U7_LP1 -> (no net)
- C17 pad 2: GND -> (no net)
- C18 pad 1: U8_LP1 -> (no net)
- C18 pad 2: GND -> (no net)
- C19 pad 1: V9 -> (no net)
- C19 pad 2: GND -> (no net)
- C2 pad 1: XLR_COLD -> (no net)
- C2 pad 2: GND -> (no net)
- C20 pad 1: U3A_OUT -> (no net)
- C20 pad 2: HEADS -> (no net)
- C21 pad 1: U2A_INM -> (no net)
- C21 pad 2: N4V5 -> (no net)
- C22 pad 1: V5 -> (no net)
- C22 pad 2: GND -> (no net)
- C23 pad 1: V9 -> (no net)
- C23 pad 2: GND -> (no net)
- C24 pad 1: VEE -> (no net)
- C24 pad 2: GND -> (no net)
- C25 pad 1: U1_OA -> (no net)
- C25 pad 2: U1_BP -> (no net)
- C26 pad 1: NOISE_D -> (no net)
- C26 pad 2: NOISE_MIX -> (no net)
- C27 pad 1: PRE_W -> (no net)
- C27 pad 2: FALA -> (no net)
- C28 pad 1: SHAPE -> (no net)
- C28 pad 2: FILT_SW -> (no net)
- C29 pad 1: WET_MIX -> (no net)
- C29 pad 2: LE_IN -> (no net)
- C3 pad 1: WET_LP -> (no net)
- C3 pad 2: GND -> (no net)
- C30 pad 1: MIX -> (no net)
- C30 pad 2: EQ_IN -> (no net)
- C31 pad 1: V5 -> (no net)
- C31 pad 2: GND -> (no net)
- C32 pad 1: V5 -> (no net)
- C32 pad 2: GND -> (no net)
- C33 pad 1: V5 -> (no net)
- C33 pad 2: GND -> (no net)
- C34 pad 1: U6_OUT -> (no net)
- C34 pad 2: U6_SW -> (no net)
- C35 pad 1: U7_OUT -> (no net)
- C35 pad 2: U7_SW -> (no net)
- C36 pad 1: U8_OUT -> (no net)
- C36 pad 2: U8_SW -> (no net)
- C37 pad 1: PT_REF_U6 -> (no net)
- C37 pad 2: GND -> (no net)
- C38 pad 1: PT_REF_U7 -> (no net)
- C38 pad 2: GND -> (no net)
- C39 pad 1: PT_REF_U8 -> (no net)
- C39 pad 2: GND -> (no net)
- C4 pad 1: U3A_IN -> (no net)
- C4 pad 2: U3A_OUT -> (no net)
- C40 pad 1: V9 -> (no net)
- C40 pad 2: GND -> (no net)
- C41 pad 1: PRE_W -> (no net)
- C41 pad 2: OSCIN_CW -> (no net)
- C42 pad 1: U1_OB -> (no net)
- C42 pad 2: PRE_CW -> (no net)
- C43 pad 1: LFO_D -> (no net)
- C43 pad 2: LFO_N1 -> (no net)
- C44 pad 1: LFO_N1 -> (no net)
- C44 pad 2: LFO_N2 -> (no net)
- C45 pad 1: INST_TIP -> (no net)
- C45 pad 2: EXT_IN -> (no net)
- C46 pad 1: TREM_A -> (no net)
- C46 pad 2: LFO_G -> (no net)
- C47 pad 1: VCF -> (no net)
- C47 pad 2: GND -> (no net)
- C48 pad 1: GRAVA_IN -> (no net)
- C48 pad 2: NAB_MID -> (no net)
- C49 pad 1: NAB_BASS -> (no net)
- C49 pad 2: WET -> (no net)
- C5 pad 1: U3B_IN -> (no net)
- C5 pad 2: WET -> (no net)
- C50 pad 1: VCF -> (no net)
- C50 pad 2: VCA_D -> (no net)
- C51 pad 1: U2A_OUT -> (no net)
- C51 pad 2: SW_A -> (no net)
- C52 pad 1: U2B_OUT -> (no net)
- C52 pad 2: SW_B -> (no net)
- C53 pad 1: LFO_D -> (no net)
- C53 pad 2: LFO_AC -> (no net)
- C54 pad 1: VCA_S -> (no net)
- C54 pad 2: DRY -> (no net)
- C55 pad 1: CLK_B -> (no net)
- C55 pad 2: GND -> (no net)
- C56 pad 1: U4_CAP+ -> (no net)
- C56 pad 2: U4_CAP- -> (no net)
- C57 pad 1: VEE -> (no net)
- C57 pad 2: GND -> (no net)
- C58 pad 1: V5 -> (no net)
- C58 pad 2: GND -> (no net)
- C59 pad 1: XLR_HOT -> (no net)
- C59 pad 2: PRE_R12 -> (no net)
- C6 pad 1: U2B_INM -> (no net)
- C6 pad 2: N4V5 -> (no net)
- C60 pad 1: XLR_COLD -> (no net)
- C60 pad 2: PRE_R13 -> (no net)
- C61 pad 1: V9 -> (no net)
- C61 pad 2: GND -> (no net)
- C62 pad 1: VEE -> (no net)
- C62 pad 2: GND -> (no net)
- C63 pad 1: V5 -> (no net)
- C63 pad 2: GND -> (no net)
- C64 pad 1: V9 -> (no net)
- C64 pad 2: GND -> (no net)
- C65 pad 1: VEE -> (no net)
- C65 pad 2: GND -> (no net)
- C66 pad 1: N4V5 -> (no net)
- C66 pad 2: GND -> (no net)
- C67 pad 1: N1V8 -> (no net)
- C67 pad 2: GND -> (no net)
- C68 pad 1: ENV -> (no net)
- C68 pad 2: GND -> (no net)
- C69 pad 1: U7_OUT -> (no net)
- C69 pad 2: U7_SW -> (no net)
- C7 pad 1: U6_CC1 -> (no net)
- C7 pad 2: U6_CC0 -> (no net)
- C70 pad 1: U8_OUT -> (no net)
- C70 pad 2: U8_SW -> (no net)
- C71 pad 1: TREM_B -> (no net)
- C71 pad 2: LFO_G -> (no net)
- C8 pad 1: U7_CC1 -> (no net)
- C8 pad 2: U7_CC0 -> (no net)
- C9 pad 1: U8_CC1 -> (no net)
- C9 pad 2: U8_CC0 -> (no net)
- D1 pad 1: V9 -> (no net)
- D1 pad 2: P4_TIP -> (no net)
- D2 pad 1: ENV -> (no net)
- D2 pad 2: GATE -> (no net)
- D3 pad 1: ENV -> (no net)
- D3 pad 2: FALA_A -> (no net)
- D4 pad 1: CLK_B -> (no net)
- D4 pad 2: CLK_A -> (no net)
- D6 pad 1: GND -> (no net)
- D6 pad 2: SHAPE -> (no net)
- D7 pad 1: GND -> (no net)
- D7 pad 2: WET -> (no net)
- J1 pad 1: OSC_A_POT -> (no net)
- J1 pad 10: GND -> (no net)
- J1 pad 11: N1V8 -> (no net)
- J1 pad 12: CUT_W -> (no net)
- J1 pad 13: GND -> (no net)
- J1 pad 14: SW_A -> (no net)
- J1 pad 15: SW_A_ON -> (no net)
- J1 pad 16: SW_B -> (no net)
- J1 pad 17: SW_B_ON -> (no net)
- J1 pad 18: N1V8 -> (no net)
- J1 pad 19: ENV -> (no net)
- J1 pad 2: U2A_INM -> (no net)
- J1 pad 3: OSC_B_POT -> (no net)
- J1 pad 4: U2B_INM -> (no net)
- J1 pad 5: SUM -> (no net)
- J1 pad 6: AMT_W -> (no net)
- J1 pad 7: GND -> (no net)
- J1 pad 8: EQ_OUT -> (no net)
- J1 pad 9: SHAPE_W -> (no net)
- J2 pad 1: RATE_W -> (no net)
- J2 pad 10: DEPTH_W -> (no net)
- J2 pad 11: PITCH_CV -> (no net)
- J2 pad 12: TIME_CV -> (no net)
- J2 pad 2: RATE_W -> (no net)
- J2 pad 3: GND -> (no net)
- J2 pad 4: LFO_OUT -> (no net)
- J2 pad 5: DEPTH_W -> (no net)
- J2 pad 6: GND -> (no net)
- J2 pad 7: LFO_N2 -> (no net)
- J2 pad 8: TREM_A -> (no net)
- J2 pad 9: TREM_B -> (no net)
- J3 pad 1: V5 -> (no net)
- J3 pad 10: GND -> (no net)
- J3 pad 11: STAR -> (no net)
- J3 pad 12: FB_CW -> (no net)
- J3 pad 13: DRY -> (no net)
- J3 pad 14: WET_W -> (no net)
- J3 pad 15: WET -> (no net)
- J3 pad 16: U6_SW -> (no net)
- J3 pad 17: U7_IN -> (no net)
- J3 pad 18: GND -> (no net)
- J3 pad 19: OUT -> (no net)
- J3 pad 2: TIME_W -> (no net)
- J3 pad 20: WET_W -> (no net)
- J3 pad 3: GND -> (no net)
- J3 pad 4: U6_SW -> (no net)
- J3 pad 5: H1_ON -> (no net)
- J3 pad 6: U7_SW -> (no net)
- J3 pad 7: H2_ON -> (no net)
- J3 pad 8: U8_SW -> (no net)
- J3 pad 9: H3_ON -> (no net)
- J4 pad 1: SW_A_ON -> (no net)
- J4 pad 10: FILT_TIP -> (no net)
- J4 pad 11: FILT_SW -> (no net)
- J4 pad 12: GND -> (no net)
- J4 pad 13: FCV -> (no net)
- J4 pad 15: GND -> (no net)
- J4 pad 16: VCV -> (no net)
- J4 pad 18: GND -> (no net)
- J4 pad 3: GND -> (no net)
- J4 pad 4: SW_B_ON -> (no net)
- J4 pad 6: GND -> (no net)
- J4 pad 7: EXT_IN -> (no net)
- J4 pad 9: GND -> (no net)
- J5 pad 1: LFO_OUT -> (no net)
- J5 pad 10: PRE_W -> (no net)
- J5 pad 12: GND -> (no net)
- J5 pad 13: STAR -> (no net)
- J5 pad 14: PRE_W -> (no net)
- J5 pad 15: GND -> (no net)
- J5 pad 3: GND -> (no net)
- J5 pad 4: TIME_CV -> (no net)
- J5 pad 6: GND -> (no net)
- J5 pad 7: CLK_TIP -> (no net)
- J5 pad 9: GND -> (no net)
- J6 pad 1: LED_A -> (no net)
- J6 pad 2: GND -> (no net)
- J6 pad 3: P4_TIP -> (no net)
- J6 pad 4: GND -> (no net)
- J6 pad 5: GATE -> (no net)
- J6 pad 6: GND -> (no net)
- J7 pad 1: XLR_HOT -> (no net)
- J7 pad 10: MIX -> (no net)
- J7 pad 11: OSCIN_CW -> (no net)
- J7 pad 2: XLR_COLD -> (no net)
- J7 pad 3: GND -> (no net)
- J7 pad 4: INST_TIP -> (no net)
- J7 pad 5: GND -> (no net)
- J7 pad 6: GND -> (no net)
- J7 pad 7: PRE_W -> (no net)
- J7 pad 8: PRE_CW -> (no net)
- J7 pad 9: AMT_W -> (no net)
- J8 pad 1: XLR_OUT -> (no net)
- J8 pad 2: J8_COLD -> (no net)
- J8 pad 3: GND -> (no net)
- J8 pad 4: OUT -> (no net)
- J8 pad 5: GND -> (no net)
- Q1 pad 1: U2A_INM -> (no net)
- Q1 pad 2: Q1G -> (no net)
- Q1 pad 3: N4V5 -> (no net)
- Q2 pad 1: U2B_INM -> (no net)
- Q2 pad 2: Q2G -> (no net)
- Q2 pad 3: N4V5 -> (no net)
- Q3 pad 1: NOISE_D -> (no net)
- Q3 pad 2: Q3G -> (no net)
- Q3 pad 3: NOISE_S -> (no net)
- Q4 pad 1: VCF -> (no net)
- Q4 pad 2: Q4G -> (no net)
- Q4 pad 3: N1V8 -> (no net)
- Q5 pad 1: VCA_D -> (no net)
- Q5 pad 2: ENV -> (no net)
- Q5 pad 3: VCA_S -> (no net)
- Q6 pad 1: V9 -> (no net)
- Q6 pad 2: Q6G -> (no net)
- Q6 pad 3: Q6S -> (no net)
- Q7 pad 1: LFO_D -> (no net)
- Q7 pad 2: LFO_G -> (no net)
- Q7 pad 3: LFO_S -> (no net)
- R1 pad 1: XLR_OUT -> (no net)
- R1 pad 2: GND -> (no net)
- R10 pad 1: H3A -> (no net)
- R10 pad 2: H3B -> (no net)
- R11 pad 1: TIME_W -> (no net)
- R11 pad 2: PT6_U6 -> (no net)
- R12 pad 1: PRE_R12 -> (no net)
- R12 pad 2: U1_INP -> (no net)
- R13 pad 1: PRE_R13 -> (no net)
- R13 pad 2: U1_INM -> (no net)
- R14 pad 1: V9 -> (no net)
- R14 pad 2: LED_A -> (no net)
- R15 pad 1: LFO_G -> (no net)
- R15 pad 2: RATE_W -> (no net)
- R16 pad 1: NAB_MID -> (no net)
- R16 pad 2: U3A_IN -> (no net)
- R18 pad 1: N1V8 -> (no net)
- R18 pad 2: GND -> (no net)
- R19 pad 1: V9 -> (no net)
- R19 pad 2: N4V5 -> (no net)
- R2 pad 1: J8_COLD -> (no net)
- R2 pad 2: GND -> (no net)
- R20 pad 1: N4V5 -> (no net)
- R20 pad 2: GND -> (no net)
- R21 pad 1: U2A_OUT -> (no net)
- R21 pad 2: OSC_A_POT -> (no net)
- R22 pad 1: U2B_OUT -> (no net)
- R22 pad 2: OSC_B_POT -> (no net)
- R23 pad 1: V9 -> (no net)
- R23 pad 2: NOISE_D -> (no net)
- R24 pad 1: SW_A_ON -> (no net)
- R24 pad 2: SUM -> (no net)
- R25 pad 1: SW_B_ON -> (no net)
- R25 pad 2: SUM -> (no net)
- R26 pad 1: EXT_IN -> (no net)
- R26 pad 2: SUM -> (no net)
- R27 pad 1: EQ_OUT -> (no net)
- R27 pad 2: Q6G -> (no net)
- R28 pad 1: Q6S -> (no net)
- R28 pad 2: SHAPE -> (no net)
- R29 pad 1: SHAPE_W -> (no net)
- R29 pad 2: SHAPE -> (no net)
- R3 pad 1: NOISE_S -> (no net)
- R3 pad 2: GND -> (no net)
- R30 pad 1: FILT_TIP -> (no net)
- R30 pad 2: VCF -> (no net)
- R31 pad 1: V9 -> (no net)
- R31 pad 2: LFO_D -> (no net)
- R32 pad 1: LFO_N1 -> (no net)
- R32 pad 2: GND -> (no net)
- R33 pad 1: LFO_N2 -> (no net)
- R33 pad 2: GND -> (no net)
- R34 pad 1: VCA_S -> (no net)
- R34 pad 2: N1V8 -> (no net)
- R35 pad 1: HEADS -> (no net)
- R35 pad 2: U6_IN -> (no net)
- R36 pad 1: HEADS -> (no net)
- R36 pad 2: U7_IN -> (no net)
- R37 pad 1: HEADS -> (no net)
- R37 pad 2: U8_IN -> (no net)
- R38 pad 1: H1_ON -> (no net)
- R38 pad 2: WET_MIX -> (no net)
- R39 pad 1: H2_ON -> (no net)
- R39 pad 2: WET_MIX -> (no net)
- R4 pad 1: Q6S -> (no net)
- R4 pad 2: N4V5 -> (no net)
- R40 pad 1: H3_ON -> (no net)
- R40 pad 2: WET_MIX -> (no net)
- R41 pad 1: U6_IN -> (no net)
- R41 pad 2: U6_LP1 -> (no net)
- R42 pad 1: U1_BM -> (no net)
- R42 pad 2: U1_OB -> (no net)
- R43 pad 1: CLK_A -> (no net)
- R43 pad 2: GND -> (no net)
- R44 pad 1: OUT -> (no net)
- R44 pad 2: XLR_OUT -> (no net)
- R45 pad 1: U3B_IN -> (no net)
- R45 pad 2: NAB_BASS -> (no net)
- R46 pad 1: DRY -> (no net)
- R46 pad 2: STAR -> (no net)
- R47 pad 1: U7_IN -> (no net)
- R47 pad 2: U7_LP1 -> (no net)
- R48 pad 1: U8_IN -> (no net)
- R48 pad 2: U8_LP1 -> (no net)
- R49 pad 1: WET -> (no net)
- R49 pad 2: WET_LP -> (no net)
- R5 pad 1: LFO_S -> (no net)
- R5 pad 2: GND -> (no net)
- R50 pad 1: FALA -> (no net)
- R50 pad 2: FALA_A -> (no net)
- R51 pad 1: STAR -> (no net)
- R51 pad 2: GRAVA_IN -> (no net)
- R52 pad 1: U3A_IN -> (no net)
- R52 pad 2: U3A_OUT -> (no net)
- R53 pad 1: LE_IN -> (no net)
- R53 pad 2: U3B_IN -> (no net)
- R54 pad 1: U3B_IN -> (no net)
- R54 pad 2: WET -> (no net)
- R55 pad 1: V9 -> (no net)
- R55 pad 2: N1V8 -> (no net)
- R56 pad 1: H2B -> (no net)
- R56 pad 2: PT6_U7 -> (no net)
- R57 pad 1: U1_INM -> (no net)
- R57 pad 2: U1_OA -> (no net)
- R58 pad 1: U1_INP -> (no net)
- R58 pad 2: GND -> (no net)
- R59 pad 1: CLK_TIP -> (no net)
- R59 pad 2: CLK_A -> (no net)
- R6 pad 1: U1_BM -> (no net)
- R6 pad 2: GND -> (no net)
- R60 pad 1: H3B -> (no net)
- R60 pad 2: PT6_U8 -> (no net)
- R61 pad 1: VCF -> (no net)
- R61 pad 2: RES_W -> (no net)
- R62 pad 1: U2A_OUT -> (no net)
- R62 pad 2: U2A_INP -> (no net)
- R63 pad 1: U2A_INP -> (no net)
- R63 pad 2: N4V5 -> (no net)
- R64 pad 1: NOISE_MIX -> (no net)
- R64 pad 2: SUM -> (no net)
- R65 pad 1: PITCH_CV -> (no net)
- R65 pad 2: Q1G -> (no net)
- R66 pad 1: PITCH_CV -> (no net)
- R66 pad 2: Q2G -> (no net)
- R67 pad 1: Q4G -> (no net)
- R67 pad 2: FCV -> (no net)
- R68 pad 1: CUT_W -> (no net)
- R68 pad 2: Q4G -> (no net)
- R69 pad 1: ENV -> (no net)
- R69 pad 2: VCV -> (no net)
- R7 pad 1: TIME_W -> (no net)
- R7 pad 2: H2A -> (no net)
- R70 pad 1: CLK_B -> (no net)
- R70 pad 2: TIME_CV -> (no net)
- R71 pad 1: WET -> (no net)
- R71 pad 2: WET_W -> (no net)
- R72 pad 1: U2B_OUT -> (no net)
- R72 pad 2: U2B_INP -> (no net)
- R73 pad 1: U2B_INP -> (no net)
- R73 pad 2: N4V5 -> (no net)
- R74 pad 1: ENV -> (no net)
- R74 pad 2: GND -> (no net)
- R75 pad 1: TIME_CV -> (no net)
- R75 pad 2: PT6_U6 -> (no net)
- R76 pad 1: TIME_CV -> (no net)
- R76 pad 2: PT6_U7 -> (no net)
- R77 pad 1: TIME_CV -> (no net)
- R77 pad 2: PT6_U8 -> (no net)
- R78 pad 1: CLK_B -> (no net)
- R78 pad 2: GND -> (no net)
- R79 pad 1: LFO_AC -> (no net)
- R79 pad 2: LFO_OUT -> (no net)
- R8 pad 1: H2A -> (no net)
- R8 pad 2: H2B -> (no net)
- R80 pad 1: Q3G -> (no net)
- R80 pad 2: GND -> (no net)
- R81 pad 1: LFO_G -> (no net)
- R81 pad 2: GND -> (no net)
- R9 pad 1: TIME_W -> (no net)
- R9 pad 2: H3A -> (no net)
- RV1 pad 1: WET -> (no net)
- RV1 pad 2: FB_CW -> (no net)
- RV1 pad 3: FB_CW -> (no net)
- RV2 pad 1: FILT_TIP -> (no net)
- RV2 pad 2: RES_W -> (no net)
- RV2 pad 3: FILT_TIP -> (no net)
- U1 pad 1: U1_OA -> (no net)
- U1 pad 2: U1_INM -> (no net)
- U1 pad 3: U1_INP -> (no net)
- U1 pad 4: VEE -> (no net)
- U1 pad 5: U1_BP -> (no net)
- U1 pad 6: U1_BM -> (no net)
- U1 pad 7: U1_OB -> (no net)
- U1 pad 8: V9 -> (no net)
- U2 pad 1: U2A_OUT -> (no net)
- U2 pad 2: U2A_INM -> (no net)
- U2 pad 3: U2A_INP -> (no net)
- U2 pad 4: GND -> (no net)
- U2 pad 5: U2B_INP -> (no net)
- U2 pad 6: U2B_INM -> (no net)
- U2 pad 7: U2B_OUT -> (no net)
- U2 pad 8: V9 -> (no net)
- U3 pad 1: U3A_OUT -> (no net)
- U3 pad 2: U3A_IN -> (no net)
- U3 pad 3: GND -> (no net)
- U3 pad 4: VEE -> (no net)
- U3 pad 5: GND -> (no net)
- U3 pad 6: U3B_IN -> (no net)
- U3 pad 7: WET -> (no net)
- U3 pad 8: V9 -> (no net)
- U4 pad 2: U4_CAP+ -> (no net)
- U4 pad 3: GND -> (no net)
- U4 pad 4: U4_CAP- -> (no net)
- U4 pad 5: VEE -> (no net)
- U4 pad 8: V9 -> (no net)
- U5 pad 1: V9 -> (no net)
- U5 pad 2: GND -> (no net)
- U5 pad 3: V5 -> (no net)
- U6 pad 1: V5 -> (no net)
- U6 pad 10: U6_OP -> (no net)
- U6 pad 11: U6_OP -> (no net)
- U6 pad 12: U6_OP -> (no net)
- U6 pad 13: U6_OP -> (no net)
- U6 pad 14: U6_OUT -> (no net)
- U6 pad 15: U6_LP1 -> (no net)
- U6 pad 16: U6_IN -> (no net)
- U6 pad 2: PT_REF_U6 -> (no net)
- U6 pad 3: GND -> (no net)
- U6 pad 4: GND -> (no net)
- U6 pad 6: PT6_U6 -> (no net)
- U6 pad 7: U6_CC1 -> (no net)
- U6 pad 8: U6_CC0 -> (no net)
- U6 pad 9: U6_OP -> (no net)
- U7 pad 1: V5 -> (no net)
- U7 pad 10: U7_OP -> (no net)
- U7 pad 11: U7_OP -> (no net)
- U7 pad 12: U7_OP -> (no net)
- U7 pad 13: U7_OP -> (no net)
- U7 pad 14: U7_OUT -> (no net)
- U7 pad 15: U7_LP1 -> (no net)
- U7 pad 16: U7_IN -> (no net)
- U7 pad 2: PT_REF_U7 -> (no net)
- U7 pad 3: GND -> (no net)
- U7 pad 4: GND -> (no net)
- U7 pad 6: PT6_U7 -> (no net)
- U7 pad 7: U7_CC1 -> (no net)
- U7 pad 8: U7_CC0 -> (no net)
- U7 pad 9: U7_OP -> (no net)
- U8 pad 1: V5 -> (no net)
- U8 pad 10: U8_OP -> (no net)
- U8 pad 11: U8_OP -> (no net)
- U8 pad 12: U8_OP -> (no net)
- U8 pad 13: U8_OP -> (no net)
- U8 pad 14: U8_OUT -> (no net)
- U8 pad 15: U8_LP1 -> (no net)
- U8 pad 16: U8_IN -> (no net)
- U8 pad 2: PT_REF_U8 -> (no net)
- U8 pad 3: GND -> (no net)
- U8 pad 4: GND -> (no net)
- U8 pad 6: PT6_U8 -> (no net)
- U8 pad 7: U8_CC1 -> (no net)
- U8 pad 8: U8_CC0 -> (no net)
- U8 pad 9: U8_OP -> (no net)
- U9 pad 1: EQ_A -> (no net)
- U9 pad 2: EQ_A -> (no net)
- U9 pad 3: EQ_IN -> (no net)
- U9 pad 4: VEE -> (no net)
- U9 pad 5: EQ_A -> (no net)
- U9 pad 6: EQ_OUT -> (no net)
- U9 pad 7: EQ_OUT -> (no net)
- U9 pad 8: V9 -> (no net)
Routing:
- net GND: track 1576.4 -> 0.00 mm, vias 2 -> 0
- net V9: track 902.1 -> 0.00 mm, vias 2 -> 0
- net V5: track 636.2 -> 0.00 mm, vias 3 -> 0
- net N1V8: track 482.9 -> 0.00 mm, vias 1 -> 0
- net TIME_CV: track 459.4 -> 0.00 mm, vias 6 -> 0
- net N4V5: track 433.8 -> 0.00 mm, vias 2 -> 0
- net PRE_W: track 398.0 -> 0.00 mm, vias 4 -> 0
- net EQ_OUT: track 385.8 -> 0.00 mm
- net OUT: track 373.0 -> 0.00 mm
- net WET: track 359.4 -> 0.00 mm, vias 1 -> 0
- net VEE: track 357.3 -> 0.00 mm
- net U7_SW: track 339.8 -> 0.00 mm, vias 1 -> 0
- net SUM: track 328.6 -> 0.00 mm, vias 1 -> 0
- net EXT_IN: track 326.9 -> 0.00 mm, vias 2 -> 0
- net SW_B_ON: track 323.0 -> 0.00 mm, vias 1 -> 0
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- removed copper zone on B.Cu, net GND
Other:
- board size 300 x 300 mm -> 300 x 140 mm
- board text added: "V9 GND VEE V5 4V5 1V8"
- board text added: "VOZ-9 BASE 300 x 140 mm"
- board text removed: "VOZ-9 BASE 300 x 300 mm"
- board text removed: "barramento V9 GND VEE V5 4V5 1V8"
- board text removed: "canal de audio"
- board text removed: "fio na base, pino 1 a esquerda cobre no verso corredores livres para o barramento e o audio"

Commit message: Agrupa cada função da BASE num bloco curto com nome na seda.
OSC, VCF, VCA, LFO, NAB e as três heads seguem o sinal, não o tamanho da peça. H1, H2 e H3 repetem a mesma figura, com os resistores em pé.

Co-authored-by: Andrey <andreysenes@users.noreply.github.com>
Parts:
- moved R67 248.0 mm to (263.0, 47.8)
- moved R73 214.1 mm to (65.4, 55.0)
- moved Q4 206.6 mm to (222.3, 49.0)
- moved Q5 201.1 mm to (216.2, 102.9)
- moved R61 193.9 mm to (221.7, 55.0)
- moved RV2 193.6 mm to (240.6, 56.2)
- moved C63 192.6 mm to (245.6, 81.4)
- moved R74 190.8 mm to (251.0, 101.7)
- moved R34 186.9 mm to (223.3, 101.7)
- moved D2 186.4 mm to (227.8, 109.7)
- moved C68 186.0 mm to (243.9, 102.9)
- moved C47 184.1 mm to (241.6, 47.8)
- moved C27 182.1 mm to (240.2, 109.7)
- moved R66 180.0 mm to (87.1, 55.0)
- moved R68 173.1 mm to (251.1, 47.8)
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Other:
- board text added: "FB"
- board text added: "H1"
- board text added: "H2"
- board text added: "H3"
- board text added: "LFO"
- board text added: "NOISE"
- board text added: "SHAPE"
- board text added: "TEMPO"
- board text added: "VCA"
- board text added: "VCF"
- board text removed: "FITA"
- board text removed: "MOD"
- board text removed: "V9 GND VEE V5 4V5 1V8"
