File: voz-9/kicad/voz-9.kicad_sch (KiCad schematic)
At the start: 189 parts, among them J1 OSC, J2 LFO, J3 DELAY, J4 PATCH A, J5 PATCH B, J6 CTRL, J7 IN+PRE, J8 OUT, J9 EQ424, Q1 J201, Q2 J201, Q3 J201, Q4 J201, Q5 J201, Q6 J201, Q7 2N5457, U1 NE5532, U2 TL072, U3 TL072, U4 MAX1044, U5 78M05, U6 PT2399, U7 PT2399, U8 PT2399, U9 TL072

Commit message: Espalha os blocos na BASE e troca J1–J9 por pinos 1×N na borda de baixo.
O circuito deixa o bloco central de 220×160 e ocupa a placa de 300×300 por faixas, com folga para solda. Os conectores do painel na placa passam de soquete fêmea 2×N para barra de pinos macho; o fio solda na base.

Co-authored-by: Andrey <andreysenes@users.noreply.github.com>
Parts:
- J1, J3, J4: footprint voz9:PinSocket_2x10_TopBottom -> Connector_PinHeader_2.54mm:PinHeader_1x20_P2.54mm_Vertical; symbol Connector_Generic:Conn_02x10_Top_Bottom -> Connector_Generic:Conn_01x20
- J2, J7, J9: footprint voz9:PinSocket_2x06_TopBottom -> Connector_PinHeader_2.54mm:PinHeader_1x12_P2.54mm_Vertical; symbol Connector_Generic:Conn_02x06_Top_Bottom -> Connector_Generic:Conn_01x12
- J5: footprint voz9:PinSocket_2x08_TopBottom -> Connector_PinHeader_2.54mm:PinHeader_1x16_P2.54mm_Vertical; symbol Connector_Generic:Conn_02x08_Top_Bottom -> Connector_Generic:Conn_01x16
- J6, J8: footprint voz9:PinSocket_2x03_TopBottom -> Connector_PinHeader_2.54mm:PinHeader_1x06_P2.54mm_Vertical; symbol Connector_Generic:Conn_02x03_Top_Bottom -> Connector_Generic:Conn_01x06
Other:
- note added: "VOZ-9 BASE 300×300 mm. Blocos espalhados na placa. J1–J9 são pinos 1×N na borda de baixo; o fio entra no pino. Numeração 1…N igual à tabela de pcb.md. Ainda sem ligações. D6/D7 = MP20. Q7 2N5457: conferir a pinagem do lote."
- note removed: "VOZ-9 BASE 300×300 mm — peças do pcb.svg, ainda sem ligações. D6/D7 = MP20. J1–J9 numerados em linha (pino 1 no canto). Q7 2N5457: conferir pinagem do lote."
- moved on the sheet: J1, J2, J3, J4, J5, J6, J7, J8, J9
Changed lines of the file:
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@@
 	)
 	(symbol
-		(lib_id "Connector_Generic:Conn_02x10_Top_Bottom")
+		(lib_id "Connector_Generic:Conn_01x20")
 		(at 25.00 392.00 0)
 		(unit 1)
@@
 			(effects (font (size 1.27 1.27)) (justify left))
 		)
-		(property "Footprint" "voz9:PinSocket_2x10_TopBottom"
+		(property "Footprint" "Connector_PinHeader_2.54mm:PinHeader_1x20_P2.54mm_Vertical"
 			(at 25.00 392.00 0)
 			(hide yes)
@@
 	)
 	(symbol
-		(lib_id "Connector_Generic:Conn_02x06_Top_Bottom")
+		(lib_id "Connector_Generic:Conn_01x12")
 		(at 25.00 374.00 0)
 		(unit 1)
@@
 			(effects (font (size 1.27 1.27)) (justify left))
 		)
-		(property "Footprint" "voz9:PinSocket_2x06_TopBottom"
+		(property "Footprint" "Connector_PinHeader_2.54mm:PinHeader_1x12_P2.54mm_Vertical"
 			(at 25.00 374.00 0)
 			(hide yes)
@@
 	)
 	(symbol
-		(lib_id "Connector_Generic:Conn_02x10_Top_Bottom")
+		(lib_id "Connector_Generic:Conn_01x20")
 		(at 25.00 356.00 0)
 		(unit 1)
@@
 			(effects (font (size 1.27 1.27)) (justify left))
 		)
-		(property "Footprint" "voz9:PinSocket_2x10_TopBottom"
+		(property "Footprint" "Connector_PinHeader_2.54mm:PinHeader_1x20_P2.54mm_Vertical"
 			(at 25.00 356.00 0)
 			(hide yes)
@@
 	)
 	(symbol
-		(lib_id "Connector_Generic:Conn_02x10_Top_Bottom")
+		(lib_id "Connector_Generic:Conn_01x20")
 		(at 25.00 338.00 0)
 		(unit 1)
@@
 			(effects (font (size 1.27 1.27)) (justify left))
 		)
-		(property "Footprint" "voz9:PinSocket_2x10_TopBottom"
+		(property "Footprint" "Connector_PinHeader_2.54mm:PinHeader_1x20_P2.54mm_Vertical"
 			(at 25.00 338.00 0)
 			(hide yes)
@@
 	)
 	(symbol
-		(lib_id "Connector_Generic:Conn_02x08_Top_Bottom")
+		(lib_id "Connector_Generic:Conn_01x16")
 		(at 25.00 320.00 0)
 		(unit 1)
@@
 			(effects (font (size 1.27 1.27)) (justify left))
 		)
-		(property "Footprint" "voz9:PinSocket_2x08_TopBottom"
+		(property "Footprint" "Connector_PinHeader_2.54mm:PinHeader_1x16_P2.54mm_Vertical"
 			(at 25.00 320.00 0)
 			(hide yes)
@@
 	)
 	(symbol
-		(lib_id "Connector_Generic:Conn_02x03_Top_Bottom")
+		(lib_id "Connector_Generic:Conn_01x06")
 		(at 25.00 302.00 0)
 		(unit 1)
@@
 			(effects (font (size 1.27 1.27)) (justify left))
 		)
-		(property "Footprint" "voz9:PinSocket_2x03_TopBottom"
+		(property "Footprint" "Connector_PinHeader_2.54mm:PinHeader_1x06_P2.54mm_Vertical"
 			(at 25.00 302.00 0)
 			(hide yes)
@@
 	)
 	(symbol
-		(lib_id "Connector_Generic:Conn_02x06_Top_Bottom")
+		(lib_id "Connector_Generic:Conn_01x12")
 		(at 25.00 284.00 0)
 		(unit 1)
@@
 			(effects (font (size 1.27 1.27)) (justify left))
 		)
-		(property "Footprint" "voz9:PinSocket_2x06_TopBottom"
+		(property "Footprint" "Connector_PinHeader_2.54mm:PinHeader_1x12_P2.54mm_Vertical"
 			(at 25.00 284.00 0)
 			(hide yes)
@@
 	)
 	(symbol
-		(lib_id "Connector_Generic:Conn_02x03_Top_Bottom")
+		(lib_id "Connector_Generic:Conn_01x06")
 		(at 25.00 266.00 0)
 		(unit 1)
@@
 			(effects (font (size 1.27 1.27)) (justify left))
 		)
-		(property "Footprint" "voz9:PinSocket_2x03_TopBottom"
+		(property "Footprint" "Connector_PinHeader_2.54mm:PinHeader_1x06_P2.54mm_Vertical"
 			(at 25.00 266.00 0)
 			(hide yes)
@@
 	)
 	(symbol
-		(lib_id "Connector_Generic:Conn_02x06_Top_Bottom")
+		(lib_id "Connector_Generic:Conn_01x12")
 		(at 25.00 248.00 0)
 		(unit 1)
@@
 			(effects (font (size 1.27 1.27)) (justify left))
 		)
-		(property "Footprint" "voz9:PinSocket_2x06_TopBottom"
+		(property "Footprint" "Connector_PinHeader_2.54mm:PinHeader_1x12_P2.54mm_Vertical"
 			(at 25.00 248.00 0)
 			(hide yes)
@@
 		)
 	)
-	(text "VOZ-9 BASE 300×300 mm — peças do pcb.svg, ainda sem ligações. D6/D7 = MP20. J1–J9 numerados em linha (pino 1 no canto). Q7 2N5457: conferir pinagem do lote."
+	(text "VOZ-9 BASE 300×300 mm. Blocos espalhados na placa. J1–J9 são pinos 1×N na borda de baixo; o fio entra no pino. Numeração 1…N igual à tabela de pcb.md. Ainda sem ligações. D6/D7 = MP20. Q7 2N5457: conferir a pinagem do lote."
 		(at 20.00 408.00 0)
 		(effects (font (size 2.0 2.0)))

Commit message: Agrupa a BASE pelo sinal para encurtar trilha e jumper.
Cada bloco fica junto do conector que o serve, com corredor de alimentação em cima e de áudio no meio. O 1N5817 aponta para J6, o oscilador senta em J1 e o pré em J7. O esquema repete esses blocos, ainda sem fios.

Co-authored-by: Andrey <andreysenes@users.noreply.github.com>
Other:
- note added: "EQ"
- note added: "MOD"
- note added: "OSC"
- note added: "OUT"
- note added: "PRE"
- note added: "VOZ-9 BASE. Blocos na ordem do sinal, o mesmo agrupamento da placa. J1–J9 à esquerda de cada bloco: pino 1×N na borda de baixo da PCB. Ainda sem fios. D1 ânodo para J6. D6/D7 = MP20. Q7 2N5457: conferir a pinagem do lote. U9: baía livre para a rede do EQ."
- note removed: "CHICOTES"
- note removed: "ENV"
- note removed: "TRIM"
- note removed: "U1"
- note removed: "U2"
- note removed: "VCF"
- note removed: "VOZ-9 BASE 300×300 mm. Blocos espalhados na placa. J1–J9 são pinos 1×N na borda de baixo; o fio entra no pino. Numeração 1…N igual à tabela de pcb.md. Ainda sem ligações. D6/D7 = MP20. Q7 2N5457: conferir a pinagem do lote."
- moved on the sheet: C1, C10, C11, C12, C13, C14, C15, C16, C17, C18, C19, C2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

Commit message: Agrupa cada função da BASE num bloco curto com nome na seda.
OSC, VCF, VCA, LFO, NAB e as três heads seguem o sinal, não o tamanho da peça. H1, H2 e H3 repetem a mesma figura, com os resistores em pé.

Co-authored-by: Andrey <andreysenes@users.noreply.github.com>
Other:
- note added: "FB"
- note added: "H1"
- note added: "H2"
- note added: "H3"
- note added: "LFO"
- note added: "NOISE"
- note added: "PATCH"
- note added: "SHAPE"
- note added: "TEMPO"
- note added: "VCA"
- note added: "VCF"
- note added: "VOZ-9 BASE. Blocos curtos na ordem do sinal, o mesmo nome da seda. J1–J9 à esquerda de cada grupo: pino 1×N na borda de baixo da PCB. Ainda sem fios. D1 ânodo para J6. D6/D7 = MP20. Q7 2N5457: conferir a pinagem do lote. U9: baía livre para a rede do EQ."
- note removed: "MOD"
- note removed: "VOZ-9 BASE. Blocos na ordem do sinal, o mesmo agrupamento da placa. J1–J9 à esquerda de cada bloco: pino 1×N na borda de baixo da PCB. Ainda sem fios. D1 ânodo para J6. D6/D7 = MP20. Q7 2N5457: conferir a pinagem do lote. U9: baía livre para a rede do EQ."
- moved on the sheet: C1, C10, C11, C12, C13, C14, C15, C16, C17, C18, C19, C2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

Commit message: Tira a baía vazia do EQ na seda e encosta a fonte no U9.
O retângulo EQ 424 só reservava espaço em branco ao lado do TL072. A fonte sobe para x=106 mm, sem a caixa na seda.

Co-authored-by: Andrey <andreysenes@users.noreply.github.com>
Other:
- note added: "VOZ-9 BASE. Blocos curtos na ordem do sinal, o mesmo nome da seda. J1–J9 à esquerda de cada grupo: pino 1×N na borda de baixo da PCB. Ainda sem fios. D1 ânodo para J6. D6/D7 = MP20. Q7 2N5457: conferir a pinagem do lote."
- note removed: "VOZ-9 BASE. Blocos curtos na ordem do sinal, o mesmo nome da seda. J1–J9 à esquerda de cada grupo: pino 1×N na borda de baixo da PCB. Ainda sem fios. D1 ânodo para J6. D6/D7 = MP20. Q7 2N5457: conferir a pinagem do lote. U9: baía livre para a rede do EQ."
Changed lines of the file:
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@@
 		)
 	)
-	(text "VOZ-9 BASE. Blocos curtos na ordem do sinal, o mesmo nome da seda. J1–J9 à esquerda de cada grupo: pino 1×N na borda de baixo da PCB. Ainda sem fios. D1 ânodo para J6. D6/D7 = MP20. Q7 2N5457: conferir a pinagem do lote. U9: baía livre para a rede do EQ."
+	(text "VOZ-9 BASE. Blocos curtos na ordem do sinal, o mesmo nome da seda. J1–J9 à esquerda de cada grupo: pino 1×N na borda de baixo da PCB. Ainda sem fios. D1 ânodo para J6. D6/D7 = MP20. Q7 2N5457: conferir a pinagem do lote."
 		(at 20.00 308.00 0)
 		(effects (font (size 2.0 2.0)))

Commit message: Liga o EQ 424, o GATE e a trava do CLK como a documentação pede.
O botão GATE fica em série entre 1V8 e o ânodo do 1N4148. U9 deixa de ser
um seguidor vazio: LOW, MID e HIGH entram em J9. AMOUNT, SHAPE e DEPTH
crescem no sentido horário. R71 passa a 10 k e D5 segura o CLK em 9 V.

Co-authored-by: Andrey <andreysenes@users.noreply.github.com>
Parts:
- added C72: 100n, Capacitor_THT:C_Rect_L7.2mm_W2.5mm_P5.00mm, symbol Device:C
- added C73: 33n, Capacitor_THT:C_Rect_L7.2mm_W2.5mm_P5.00mm, symbol Device:C
- added C74: 1n, Capacitor_THT:C_Rect_L7.2mm_W2.5mm_P5.00mm, symbol Device:C
- added C75: 10n, Capacitor_THT:C_Rect_L7.2mm_W2.5mm_P5.00mm, symbol Device:C
- added D5: 1N4148, Diode_THT:D_DO-41_SOD81_P7.62mm_Horizontal, symbol Device:D
- added R82, R83, R84: 10k, Resistor_THT:R_Axial_DIN0207_L6.3mm_D2.5mm_P7.62mm_Horizontal, symbol Device:R
- added R85: 100k, Resistor_THT:R_Axial_DIN0207_L6.3mm_D2.5mm_P7.62mm_Horizontal, symbol Device:R
- added R86: 3k3, Resistor_THT:R_Axial_DIN0207_L6.3mm_D2.5mm_P7.62mm_Horizontal, symbol Device:R
- R71: value 100k -> 10k
Other:
- moved on the sheet: C10, C11, C12, C13, C14, C15, C16, C17, C18, C19, C20, C21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
